File: kicad_docs/power_and_vref.sch (KiCad schematic (older format))
At the start: 24 parts, among them J7 power_input, U1 SSM2164, U2 TL072, U3 TL072, U4 TL072, U5 TL072, U6 MAX6035xxUR50

Commit message: add AC/DC coupling caps and jumper
Parts:
- U6: footprint Package_TO_SOT_SMD:SOT-23 -> Package_TO_SOT_SMD:SOT-23_Handsoldering
Changed lines of the file:
@@
 F 0 "U6" H 1921 2296 50  0000 R CNN
 F 1 "MAX6035xxUR50" H 2750 2500 50  0000 R CNN
-F 2 "Package_TO_SOT_SMD:SOT-23" H 2250 1950 50  0001 C CIN
+F 2 "Package_TO_SOT_SMD:SOT-23_Handsoldering" H 2250 1950 50  0001 C CIN
 F 3 "https://datasheets.maximintegrated.com/en/ds/MAX6035.pdf" H 2250 1900 50  0001 C CIN
 	1    2150 2250
