File: pcb/kicad_docs/dual_VCA.kicad_pcb (KiCad board)
At the start: 2 copper layers, 45.7 x 99.1 mm, 76 parts, among them J1 signal_in_1, J2 CV_in_1, J3 signal_in_2, J4 CV_in_2, J5 signal_out_1, J6 signal_out_2, J7 power_input, J8 Conn_01x06, J9 Conn_01x06, U1 SSM2164, U2 TL072, U3 TL072, U4 TL072, U5 TL072, U6 MAX6035xxUR50

Commit message: add panel, generate interactive BOM
Other:
- board text added: "github.com/JordanAceto/Dual_2164_VCA rev 1 2020-02-23"
